File: debug.sch (KiCad schematic (older format))
At the start: 1 part, among them J16 Conn_01x03

Commit message: Add files via upload
Parts:
- removed J16: Conn_01x03, symbol Connector_Generic:Conn_01x03
- added J17: Conn_01x03, symbol Connector_Generic:Conn_01x03
Connections:
- net GND: now also J17.3 (Pin_3)
- net RX: now also J17.2 (Pin_2)
- net TX: now also J17.1 (Pin_1)
Other:
- note added: "On aura besoin d'UART pour debugger le robot, avecla possibilité de le reset\n"
- note removed: "On aura besoin d'UART :\n- pour debugger le robot\n- pour communiquer avec la f3\n"
Changed lines of the file:
@@
 $Descr A4 11693 8268
 encoding utf-8
-Sheet 22 24
+Sheet 23 24
 Title ""
 Date ""
@@
 RX
 $Comp
-L Connector_Generic:Conn_01x03 J16
-U 1 1 5E8486F8
+L Connector_Generic:Conn_01x03 J17
+U 1 1 5E88C3CE
 P 6800 2800
-F 0 "J16" H 6880 2842 50  0000 L CNN
+F 0 "J17" H 6880 2842 50  0000 L CNN
 F 1 "Conn_01x03" H 6880 2751 50  0000 L CNN
 F 2 "" H 6800 2800 50  0001 C CNN
@@
 $EndComp
 $Comp
-L power:GND #PWR0124
-U 1 1 5E8486F9
+L power:GND #PWR0125
+U 1 1 5E88DB1A
 P 6450 3100
-F 0 "#PWR0124" H 6450 2850 50  0001 C CNN
+F 0 "#PWR0125" H 6450 2850 50  0001 C CNN
 F 1 "GND" H 6455 2927 50  0000 C CNN
 F 2 "" H 6450 3100 50  0001 C CNN
@@
 Wire Wire Line
 	6450 2900 6450 3100
-Text Notes 6150 2300 0    50   ~ 0
-On aura besoin d'UART :\n- pour debugger le robot\n- pour communiquer avec la f3\n
+Text Notes 5600 2400 0    50   ~ 0
+On aura besoin d'UART pour debugger le robot, avecla possibilité de le reset\n
 $EndSCHEMATC
