File: kicad_master.sch (KiCad schematic (older format))
At the start: 8 parts, among them J1 Conn_01x02, J2 Conn_01x02

Commit message: Add files via upload
Parts:
- C3, C4: value C -> 100n
- gave numbers to parts that had none: 4
Connections:
- net +5V renamed +7.5V
Other:
- note added: "Le régulateur de tension 7V5 -> 2V8 \npour alimenter : les capteurs ToFs ; Le registre à décalage"
- note added: "Le régulateur de tension 7V5 -> 5V\npour alimenter : pont en H ; Nucleo F401RE"
- note removed: "Le régulateur de tension 7V5 -> 2V8 \npour alimenter : les capteurs ToFs"
- note removed: "Le régulateur de tension 7V5 -> 5V\npour alimenter : pont en H, pull-ups \ndes capteurs de fin de course"
