File: regulateur_7V5_2V8.sch (KiCad schematic (older format))
At the start: 5 parts, among them U3 LM317_TO3

Commit message: Add files via upload
Changed lines of the file:
@@
 $Descr A4 11693 8268
 encoding utf-8
-Sheet 13 23
+Sheet 13 22
 Title ""
 Date ""
@@
 U 1 1 5E677609
 P 5050 2900
+AR Path="/5E6772A8/5E677609" Ref="U3"  Part="1"
+AR Path="/5E8305B4/5E677609" Ref="U?"  Part="1"
 F 0 "U3" H 5050 3142 50  0000 C CNN
 F 1 "LM317_TO3" H 5050 3051 50  0000 C CNN
@@
 	4250 2900 4550 2900
 $Comp
-L power:+2V8 #PWR028
-U 1 1 5E67A02D
-P 6350 2900
-F 0 "#PWR028" H 6350 2750 50  0001 C CNN
-F 1 "+2V8" V 6365 3028 50  0000 L CNN
-F 2 "" H 6350 2900 50  0001 C CNN
-F 3 "" H 6350 2900 50  0001 C CNN
-	1    6350 2900
-	0    1    1    0
-$EndComp
-$Comp
 L Device:R R9
-U 1 1 5E67BDA8
+U 1 1 5E8486F2
 P 5500 3200
+AR Path="/5E6772A8/5E8486F2" Ref="R9"  Part="1"
+AR Path="/5E8305B4/5E8486F2" Ref="R?"  Part="1"
 F 0 "R9" H 5430 3154 50  0000 R CNN
 F 1 "240" H 5430 3245 50  0000 R CNN
@@
 $EndComp
 $Comp
-L Device:R R10
-U 1 1 5E67CD58
-P 5500 3650
-F 0 "R10" H 5430 3604 50  0000 R CNN
-F 1 "300" H 5430 3695 50  0000 R CNN
-F 2 "" V 5430 3650 50  0001 C CNN
-F 3 "~" H 5500 3650 50  0001 C CNN
-	1    5500 3650
-	-1   0    0    1
-$EndComp
-$Comp
 L Device:C C2
 U 1 1 5E67D126
 P 6050 3400
+AR Path="/5E6772A8/5E67D126" Ref="C2"  Part="1"
+AR Path="/5E8305B4/5E67D126" Ref="C?"  Part="1"
 F 0 "C2" H 6165 3446 50  0000 L CNN
 F 1 "1µ" H 6165 3355 50  0000 L CNN
@@
 U 1 1 5E67DD37
 P 4550 3450
+AR Path="/5E6772A8/5E67DD37" Ref="C1"  Part="1"
+AR Path="/5E8305B4/5E67DD37" Ref="C?"  Part="1"
 F 0 "C1" H 4665 3496 50  0000 L CNN
 F 1 "100n" H 4665 3405 50  0000 L CNN
@@
 U 1 1 5E67EDD3
 P 5100 4050
+AR Path="/5E6772A8/5E67EDD3" Ref="#PWR027"  Part="1"
+AR Path="/5E8305B4/5E67EDD3" Ref="#PWR?"  Part="1"
 F 0 "#PWR027" H 5100 3800 50  0001 C CNN
 F 1 "GND" H 5105 3877 50  0000 C CNN
@@
 Wire Wire Line
 	6050 3250 6050 2900
-Connection ~ 6050 2900
-Wire Wire Line
-	6050 2900 6350 2900
 $Comp
-L power:+7.5V #PWR?
-U 1 1 5E83FC3A
+L power:+7.5V #PWR0108
+U 1 1 5E8486F7
 P 4250 2900
-F 0 "#PWR?" H 4250 2750 50  0001 C CNN
+AR Path="/5E6772A8/5E8486F7" Ref="#PWR0108"  Part="1"
+AR Path="/5E8305B4/5E8486F7" Ref="#PWR?"  Part="1"
+F 0 "#PWR0108" H 4250 2750 50  0001 C CNN
 F 1 "+7.5V" V 4265 3028 50  0000 L CNN
 F 2 "" H 4250 2900 50  0001 C CNN
@@
 Text Notes 4200 1750 0    50   ~ 0
 Le régulateur de tension permet de convertir la tension tirée depuis\nla carte en une nouvelle tension stable.\nEn effet comme le tirage de puissance se fait via un câble, la 7V5\nde la carte alim arrivera sur le shield valant moins que 7V5 et distordu\nC'est pourquoi on tire plus de 2V8 de la carte alim et on fait\nla régulation "sur place"\n
+$Comp
+L power:+2V8 #PWR028
+U 1 1 5E67A02D
+P 6550 2900
+AR Path="/5E6772A8/5E67A02D" Ref="#PWR028"  Part="1"
+AR Path="/5E8305B4/5E67A02D" Ref="#PWR?"  Part="1"
+F 0 "#PWR028" H 6550 2750 50  0001 C CNN
+F 1 "+2V8" V 6565 3028 50  0000 L CNN
+F 2 "" H 6550 2900 50  0001 C CNN
+F 3 "" H 6550 2900 50  0001 C CNN
+	1    6550 2900
+	0    1    1    0
+$EndComp
+Connection ~ 6050 2900
+$Comp
+L Device:R R10
+U 1 1 5E67CD58
+P 5500 3650
+AR Path="/5E6772A8/5E67CD58" Ref="R10"  Part="1"
+AR Path="/5E8305B4/5E67CD58" Ref="R?"  Part="1"
+F 0 "R10" H 5430 3604 50  0000 R CNN
+F 1 "300" H 5430 3695 50  0000 R CNN
+F 2 "" V 5430 3650 50  0001 C CNN
+F 3 "~" H 5500 3650 50  0001 C CNN
+	1    5500 3650
+	-1   0    0    1
+$EndComp
+Wire Wire Line
+	6050 2900 6550 2900
 $EndSCHEMATC
