File: regulateur_7V5_3V3.sch (KiCad schematic (older format))
At the start: 5 parts, among them U3 LM317_TO3

Commit message: Add files via upload
Parts:
- R10: value 300 -> 2k
- R9: value 240 -> 1.2k
Connections:
- net +2V8 renamed +3V3
Other:
- note added: "Le régulateur de tension permet de convertir la tension tirée depuis\nla carte en une nouvelle tension stable.\nEn effet comme le tirage de puissance se fait via un câble, la 7V5\nde la carte alim arrivera sur le shield valant moins que 7V5 et distordu\nC'est pourquoi on tire plus de 3V3 de la carte alim et on fait\nla régulation "sur place"\n"
- note removed: "Le régulateur de tension permet de convertir la tension tirée depuis\nla carte en une nouvelle tension stable.\nEn effet comme le tirage de puissance se fait via un câble, la 7V5\nde la carte alim arrivera sur le shield valant moins que 7V5 et distordu\nC'est pourquoi on tire plus de 2V8 de la carte alim et on fait\nla régulation "sur place"\n"
Changed lines of the file:
@@
 $Descr A4 11693 8268
 encoding utf-8
-Sheet 13 24
+Sheet 24 24
 Title ""
 Date ""
@@
 $Comp
 L Regulator_Linear:LM317_TO3 U3
-U 1 1 5E677609
+U 1 1 5E8486F1
 P 5050 2900
-AR Path="/5E6772A8/5E677609" Ref="U3"  Part="1"
-AR Path="/5E8305B4/5E677609" Ref="U?"  Part="1"
-F 0 "U3" H 5050 3142 50  0000 C CNN
+AR Path="/5E6772A8/5E8486F1" Ref="U3"  Part="1"
+AR Path="/5E8305B4/5E8486F1" Ref="U7"  Part="1"
+F 0 "U7" H 5050 3142 50  0000 C CNN
 F 1 "LM317_TO3" H 5050 3051 50  0000 C CNN
 F 2 "Package_TO_SOT_THT:TO-3" H 5050 3100 50  0001 C CIN
@@
 $Comp
 L Device:R R9
-U 1 1 5E8486F2
+U 1 1 5E67BDA8
 P 5500 3200
-AR Path="/5E6772A8/5E8486F2" Ref="R9"  Part="1"
-AR Path="/5E8305B4/5E8486F2" Ref="R?"  Part="1"
-F 0 "R9" H 5430 3154 50  0000 R CNN
-F 1 "240" H 5430 3245 50  0000 R CNN
+AR Path="/5E6772A8/5E67BDA8" Ref="R9"  Part="1"
+AR Path="/5E8305B4/5E67BDA8" Ref="R18"  Part="1"
+F 0 "R18" H 5430 3154 50  0000 R CNN
+F 1 "1.2k" H 5430 3245 50  0000 R CNN
 F 2 "" V 5430 3200 50  0001 C CNN
 F 3 "~" H 5500 3200 50  0001 C CNN
@@
 $EndComp
 $Comp
+L Device:R R10
+U 1 1 5E8486F3
+P 5500 3650
+AR Path="/5E6772A8/5E8486F3" Ref="R10"  Part="1"
+AR Path="/5E8305B4/5E8486F3" Ref="R19"  Part="1"
+F 0 "R19" H 5430 3604 50  0000 R CNN
+F 1 "2k" H 5430 3695 50  0000 R CNN
+F 2 "" V 5430 3650 50  0001 C CNN
+F 3 "~" H 5500 3650 50  0001 C CNN
+	1    5500 3650
+	-1   0    0    1
+$EndComp
+$Comp
 L Device:C C2
-U 1 1 5E67D126
+U 1 1 5E8486F4
 P 6050 3400
-AR Path="/5E6772A8/5E67D126" Ref="C2"  Part="1"
-AR Path="/5E8305B4/5E67D126" Ref="C?"  Part="1"
-F 0 "C2" H 6165 3446 50  0000 L CNN
+AR Path="/5E6772A8/5E8486F4" Ref="C2"  Part="1"
+AR Path="/5E8305B4/5E8486F4" Ref="C11"  Part="1"
+F 0 "C11" H 6165 3446 50  0000 L CNN
 F 1 "1µ" H 6165 3355 50  0000 L CNN
 F 2 "" H 6088 3250 50  0001 C CNN
@@
 $Comp
 L Device:C C1
-U 1 1 5E67DD37
+U 1 1 5E8486F5
 P 4550 3450
-AR Path="/5E6772A8/5E67DD37" Ref="C1"  Part="1"
-AR Path="/5E8305B4/5E67DD37" Ref="C?"  Part="1"
-F 0 "C1" H 4665 3496 50  0000 L CNN
+AR Path="/5E6772A8/5E8486F5" Ref="C1"  Part="1"
+AR Path="/5E8305B4/5E8486F5" Ref="C10"  Part="1"
+F 0 "C10" H 4665 3496 50  0000 L CNN
 F 1 "100n" H 4665 3405 50  0000 L CNN
 F 2 "" H 4588 3300 50  0001 C CNN
@@
 $Comp
 L power:GND #PWR027
-U 1 1 5E67EDD3
+U 1 1 5E8486F6
 P 5100 4050
-AR Path="/5E6772A8/5E67EDD3" Ref="#PWR027"  Part="1"
-AR Path="/5E8305B4/5E67EDD3" Ref="#PWR?"  Part="1"
-F 0 "#PWR027" H 5100 3800 50  0001 C CNN
+AR Path="/5E6772A8/5E8486F6" Ref="#PWR027"  Part="1"
+AR Path="/5E8305B4/5E8486F6" Ref="#PWR0126"  Part="1"
+F 0 "#PWR0126" H 5100 3800 50  0001 C CNN
 F 1 "GND" H 5105 3877 50  0000 C CNN
 F 2 "" H 5100 4050 50  0001 C CNN
@@
 	6050 3250 6050 2900
 $Comp
-L power:+7.5V #PWR0108
-U 1 1 5E8486F7
+L power:+7.5V #PWR?
+U 1 1 5E83FC3A
 P 4250 2900
-AR Path="/5E6772A8/5E8486F7" Ref="#PWR0108"  Part="1"
-AR Path="/5E8305B4/5E8486F7" Ref="#PWR?"  Part="1"
-F 0 "#PWR0108" H 4250 2750 50  0001 C CNN
+AR Path="/5E6772A8/5E83FC3A" Ref="#PWR?"  Part="1"
+AR Path="/5E8305B4/5E83FC3A" Ref="#PWR0127"  Part="1"
+F 0 "#PWR0127" H 4250 2750 50  0001 C CNN
 F 1 "+7.5V" V 4265 3028 50  0000 L CNN
 F 2 "" H 4250 2900 50  0001 C CNN
@@
 R1\n
 Text Notes 4200 1750 0    50   ~ 0
-Le régulateur de tension permet de convertir la tension tirée depuis\nla carte en une nouvelle tension stable.\nEn effet comme le tirage de puissance se fait via un câble, la 7V5\nde la carte alim arrivera sur le shield valant moins que 7V5 et distordu\nC'est pourquoi on tire plus de 2V8 de la carte alim et on fait\nla régulation "sur place"\n
+Le régulateur de tension permet de convertir la tension tirée depuis\nla carte en une nouvelle tension stable.\nEn effet comme le tirage de puissance se fait via un câble, la 7V5\nde la carte alim arrivera sur le shield valant moins que 7V5 et distordu\nC'est pourquoi on tire plus de 3V3 de la carte alim et on fait\nla régulation "sur place"\n
 $Comp
-L power:+2V8 #PWR028
-U 1 1 5E67A02D
-P 6550 2900
-AR Path="/5E6772A8/5E67A02D" Ref="#PWR028"  Part="1"
-AR Path="/5E8305B4/5E67A02D" Ref="#PWR?"  Part="1"
-F 0 "#PWR028" H 6550 2750 50  0001 C CNN
-F 1 "+2V8" V 6565 3028 50  0000 L CNN
-F 2 "" H 6550 2900 50  0001 C CNN
-F 3 "" H 6550 2900 50  0001 C CNN
-	1    6550 2900
+L power:+3V3 #PWR0128
+U 1 1 5E833694
+P 6450 2900
+F 0 "#PWR0128" H 6450 2750 50  0001 C CNN
+F 1 "+3V3" V 6465 3028 50  0000 L CNN
+F 2 "" H 6450 2900 50  0001 C CNN
+F 3 "" H 6450 2900 50  0001 C CNN
+	1    6450 2900
 	0    1    1    0
 $EndComp
 Wire Wire Line
-	6050 2900 6550 2900
+	6050 2900 6450 2900
 Connection ~ 6050 2900
-$Comp
-L Device:R R10
-U 1 1 5E67CD58
-P 5500 3650
-AR Path="/5E6772A8/5E67CD58" Ref="R10"  Part="1"
-AR Path="/5E8305B4/5E67CD58" Ref="R?"  Part="1"
-F 0 "R10" H 5430 3604 50  0000 R CNN
-F 1 "300" H 5430 3695 50  0000 R CNN
-F 2 "" V 5430 3650 50  0001 C CNN
-F 3 "~" H 5500 3650 50  0001 C CNN
-	1    5500 3650
-	-1   0    0    1
-$EndComp
 $EndSCHEMATC
