File: regulateur_7V5_5V.sch (KiCad schematic (older format))
At the start: 5 parts

Commit message: Add files via upload
Parts:
- gave numbers to parts that had none: 5
Changed lines of the file:
@@
 $Descr A4 11693 8268
 encoding utf-8
-Sheet 20 23
+Sheet 20 22
 Title ""
 Date ""
@@
 P 4850 2900
 AR Path="/5E6772A8/5E84323B" Ref="U?"  Part="1"
-AR Path="/5E83D769/5E84323B" Ref="U?"  Part="1"
-F 0 "U?" H 4850 3142 50  0000 C CNN
+AR Path="/5E83D769/5E84323B" Ref="U6"  Part="1"
+F 0 "U6" H 4850 3142 50  0000 C CNN
 F 1 "LM317_TO3" H 4850 3051 50  0000 C CNN
 F 2 "Package_TO_SOT_THT:TO-3" H 4850 3100 50  0001 C CIN
@@
 P 5300 3200
 AR Path="/5E6772A8/5E84324E" Ref="R?"  Part="1"
-AR Path="/5E83D769/5E84324E" Ref="R?"  Part="1"
-F 0 "R?" H 5230 3154 50  0000 R CNN
+AR Path="/5E83D769/5E84324E" Ref="R16"  Part="1"
+F 0 "R16" H 5230 3154 50  0000 R CNN
 F 1 "1k" H 5230 3245 50  0000 R CNN
 F 2 "" V 5230 3200 50  0001 C CNN
@@
 P 5300 3650
 AR Path="/5E6772A8/5E843254" Ref="R?"  Part="1"
-AR Path="/5E83D769/5E843254" Ref="R?"  Part="1"
-F 0 "R?" H 5230 3604 50  0000 R CNN
+AR Path="/5E83D769/5E843254" Ref="R17"  Part="1"
+F 0 "R17" H 5230 3604 50  0000 R CNN
 F 1 "3k" H 5230 3695 50  0000 R CNN
 F 2 "" V 5230 3650 50  0001 C CNN
@@
 P 5850 3400
 AR Path="/5E6772A8/5E84325A" Ref="C?"  Part="1"
-AR Path="/5E83D769/5E84325A" Ref="C?"  Part="1"
-F 0 "C?" H 5965 3446 50  0000 L CNN
+AR Path="/5E83D769/5E84325A" Ref="C9"  Part="1"
+F 0 "C9" H 5965 3446 50  0000 L CNN
 F 1 "1µ" H 5965 3355 50  0000 L CNN
 F 2 "" H 5888 3250 50  0001 C CNN
@@
 P 4350 3450
 AR Path="/5E6772A8/5E843260" Ref="C?"  Part="1"
-AR Path="/5E83D769/5E843260" Ref="C?"  Part="1"
-F 0 "C?" H 4465 3496 50  0000 L CNN
+AR Path="/5E83D769/5E843260" Ref="C8"  Part="1"
+F 0 "C8" H 4465 3496 50  0000 L CNN
 F 1 "100n" H 4465 3405 50  0000 L CNN
 F 2 "" H 4388 3300 50  0001 C CNN
@@
 P 4900 4050
 AR Path="/5E6772A8/5E843278" Ref="#PWR?"  Part="1"
-AR Path="/5E83D769/5E843278" Ref="#PWR?"  Part="1"
-F 0 "#PWR?" H 4900 3800 50  0001 C CNN
+AR Path="/5E83D769/5E843278" Ref="#PWR0119"  Part="1"
+F 0 "#PWR0119" H 4900 3800 50  0001 C CNN
 F 1 "GND" H 4905 3877 50  0000 C CNN
 F 2 "" H 4900 4050 50  0001 C CNN
@@
 Wire Wire Line
 	5850 3250 5850 2900
-Connection ~ 5850 2900
-Wire Wire Line
-	5850 2900 6150 2900
 $Comp
-L power:+7.5V #PWR?
+L power:+7.5V #PWR0120
 U 1 1 5E8435B8
 P 4050 2900
-F 0 "#PWR?" H 4050 2750 50  0001 C CNN
+F 0 "#PWR0120" H 4050 2750 50  0001 C CNN
 F 1 "+7.5V" V 4065 3028 50  0000 L CNN
 F 2 "" H 4050 2900 50  0001 C CNN
@@
 $EndComp
 $Comp
-L power:+5V #PWR?
+L power:+5V #PWR0121
 U 1 1 5E8445EA
-P 6150 2900
-F 0 "#PWR?" H 6150 2750 50  0001 C CNN
-F 1 "+5V" V 6165 3028 50  0000 L CNN
-F 2 "" H 6150 2900 50  0001 C CNN
-F 3 "" H 6150 2900 50  0001 C CNN
-	1    6150 2900
+P 6250 2900
+F 0 "#PWR0121" H 6250 2750 50  0001 C CNN
+F 1 "+5V" V 6265 3028 50  0000 L CNN
+F 2 "" H 6250 2900 50  0001 C CNN
+F 3 "" H 6250 2900 50  0001 C CNN
+	1    6250 2900
 	0    1    1    0
 $EndComp
@@
 Wire Notes Line
 	4200 4400 6100 4400
+Wire Wire Line
+	5850 2900 6250 2900
+Connection ~ 5850 2900
 $EndSCHEMATC
