File: Conn_ToF.sch (KiCad schematic (older format))
At the start: 1 part, among them J3 Conn_01x05

Commit message: Add files via upload
Other:
- note added: "Les capteurs ToFs (Time of Flight) permettent de mesurer la\ndistance à l'objet en face d'eux de manière plus précise\nque les capteurs ultrason, moyennant une mise en place\nun peu plus compliquée\nIls communiquent avec la F4 via protocole I2C"
- note removed: "Les capteurs ToFs (Time of Flight) permettent de mesure la\ndistance à l'objet en face d'eux de manière plus précise\nque les capteurs ultrason, moyennant une mise en place\nun peu plus compliquée\nIls communiquent avec la F4 via protocole I2C"
Changed lines of the file:
@@
 $Descr A4 11693 8268
 encoding utf-8
-Sheet 3 23
+Sheet 3 22
 Title ""
 Date ""
@@
 AR Path="/5E68B664/5E684EEF" Ref="J9"  Part="1"
 AR Path="/5E68B669/5E684EEF" Ref="J10"  Part="1"
-F 0 "J3" H 5330 3492 50  0000 L CNN
+F 0 "J10" H 5330 3492 50  0000 L CNN
 F 1 "Conn_01x05" H 5330 3401 50  0000 L CNN
 F 2 "" H 5250 3450 50  0001 C CNN
@@
 AR Path="/5E68B664/5E6859B3" Ref="#PWR019"  Part="1"
 AR Path="/5E68B669/5E6859B3" Ref="#PWR021"  Part="1"
-F 0 "#PWR07" H 4900 3400 50  0001 C CNN
+F 0 "#PWR021" H 4900 3400 50  0001 C CNN
 F 1 "GND" V 4905 3522 50  0000 R CNN
 F 2 "" H 4900 3650 50  0001 C CNN
@@
 AR Path="/5E68B664/5E686310" Ref="#PWR018"  Part="1"
 AR Path="/5E68B669/5E686310" Ref="#PWR020"  Part="1"
-F 0 "#PWR06" H 4900 3100 50  0001 C CNN
+F 0 "#PWR020" H 4900 3100 50  0001 C CNN
 F 1 "+2V8" V 4915 3378 50  0000 L CNN
 F 2 "" H 4900 3250 50  0001 C CNN
@@
 	4900 3650 5050 3650
 Text Notes 4100 2700 0    50   ~ 0
-Les capteurs ToFs (Time of Flight) permettent de mesure la\ndistance à l'objet en face d'eux de manière plus précise\nque les capteurs ultrason, moyennant une mise en place\nun peu plus compliquée\nIls communiquent avec la F4 via protocole I2C
+Les capteurs ToFs (Time of Flight) permettent de mesurer la\ndistance à l'objet en face d'eux de manière plus précise\nque les capteurs ultrason, moyennant une mise en place\nun peu plus compliquée\nIls communiquent avec la F4 via protocole I2C
 $EndSCHEMATC

Commit message: Add files via upload
Parts:
- J3: value Conn_01x05 -> ToF; footprint (none) -> Connector_JST:JST_PH_B5B-PH-K_1x05_P2.00mm_Vertical
Changed lines of the file:
@@
 EESchema Schematic File Version 4
-LIBS:kicad_master-cache
 EELAYER 30 0
 EELAYER END
 $Descr A4 11693 8268
 encoding utf-8
-Sheet 3 22
+Sheet 4 21
 Title ""
 Date ""
@@
 AR Path="/5E68B664/5E684EEF" Ref="J9"  Part="1"
 AR Path="/5E68B669/5E684EEF" Ref="J10"  Part="1"
-F 0 "J10" H 5330 3492 50  0000 L CNN
-F 1 "Conn_01x05" H 5330 3401 50  0000 L CNN
-F 2 "" H 5250 3450 50  0001 C CNN
+F 0 "J4" H 5330 3492 50  0000 L CNN
+F 1 "ToF" H 5330 3401 50  0000 L CNN
+F 2 "Connector_JST:JST_PH_B5B-PH-K_1x05_P2.00mm_Vertical" H 5250 3450 50  0001 C CNN
 F 3 "~" H 5250 3450 50  0001 C CNN
 	1    5250 3450
@@
 AR Path="/5E68B664/5E6859B3" Ref="#PWR019"  Part="1"
 AR Path="/5E68B669/5E6859B3" Ref="#PWR021"  Part="1"
-F 0 "#PWR021" H 4900 3400 50  0001 C CNN
+F 0 "#PWR09" H 4900 3400 50  0001 C CNN
 F 1 "GND" V 4905 3522 50  0000 R CNN
 F 2 "" H 4900 3650 50  0001 C CNN
@@
 AR Path="/5E68B664/5E686310" Ref="#PWR018"  Part="1"
 AR Path="/5E68B669/5E686310" Ref="#PWR020"  Part="1"
-F 0 "#PWR020" H 4900 3100 50  0001 C CNN
+F 0 "#PWR08" H 4900 3100 50  0001 C CNN
 F 1 "+2V8" V 4915 3378 50  0000 L CNN
 F 2 "" H 4900 3250 50  0001 C CNN

Commit message: avancement général du routage
Parts:
- J3: symbol Connector_Generic:Conn_01x05 -> shield_etage2-rescue:Conn_01x05-Connector_Generic
Changed lines of the file:
@@
 $Descr A4 11693 8268
 encoding utf-8
-Sheet 4 21
+Sheet 8 21
 Title ""
 Date ""
@@
 $EndDescr
 $Comp
-L Connector_Generic:Conn_01x05 J3
+L shield_etage2-rescue:Conn_01x05-Connector_Generic J3
 U 1 1 5E684EEF
 P 5250 3450
@@
 AR Path="/5E68B664/5E684EEF" Ref="J9"  Part="1"
 AR Path="/5E68B669/5E684EEF" Ref="J10"  Part="1"
-F 0 "J4" H 5330 3492 50  0000 L CNN
+F 0 "J8" H 5330 3492 50  0000 L CNN
 F 1 "ToF" H 5330 3401 50  0000 L CNN
 F 2 "Connector_JST:JST_PH_B5B-PH-K_1x05_P2.00mm_Vertical" H 5250 3450 50  0001 C CNN
@@
 $EndComp
 $Comp
-L power:GND #PWR07
+L shield_etage2-rescue:GND-power #PWR07
 U 1 1 5E6859B3
 P 4900 3650
@@
 AR Path="/5E68B664/5E6859B3" Ref="#PWR019"  Part="1"
 AR Path="/5E68B669/5E6859B3" Ref="#PWR021"  Part="1"
-F 0 "#PWR09" H 4900 3400 50  0001 C CNN
+F 0 "#PWR017" H 4900 3400 50  0001 C CNN
 F 1 "GND" V 4905 3522 50  0000 R CNN
 F 2 "" H 4900 3650 50  0001 C CNN
@@
 $EndComp
 $Comp
-L power:+2V8 #PWR06
+L shield_etage2-rescue:+2V8-power #PWR06
 U 1 1 5E686310
 P 4900 3250
@@
 AR Path="/5E68B664/5E686310" Ref="#PWR018"  Part="1"
 AR Path="/5E68B669/5E686310" Ref="#PWR020"  Part="1"
-F 0 "#PWR08" H 4900 3100 50  0001 C CNN
+F 0 "#PWR016" H 4900 3100 50  0001 C CNN
 F 1 "+2V8" V 4915 3378 50  0000 L CNN
 F 2 "" H 4900 3250 50  0001 C CNN
