File: Conn_ToF.sch (KiCad schematic (older format))
At the start: 1 part, among them J3 ToF

Commit message: addition of second motor and ArUco outputs, note the last edition is the one called gange
Changed lines of the file:
@@
 AR Path="/5E68B664/5E684EEF" Ref="J9"  Part="1"
 AR Path="/5E68B669/5E684EEF" Ref="J10"  Part="1"
-F 0 "J10" H 5330 3492 50  0000 L CNN
+F 0 "J3" H 5330 3492 50  0000 L CNN
 F 1 "ToF" H 5330 3401 50  0000 L CNN
 F 2 "Connector_JST:JST_PH_B5B-PH-K_1x05_P2.00mm_Vertical" H 5250 3450 50  0001 C CNN
@@
 AR Path="/5E68B664/5E6859B3" Ref="#PWR022"  Part="1"
 AR Path="/5E68B669/5E6859B3" Ref="#PWR024"  Part="1"
-F 0 "#PWR024" H 4900 3400 50  0001 C CNN
+F 0 "#PWR010" H 4900 3400 50  0001 C CNN
 F 1 "GND" V 4905 3522 50  0000 R CNN
 F 2 "" H 4900 3650 50  0001 C CNN
@@
 AR Path="/5E68B669/5E686310" Ref="#PWR023"  Part="1"
 AR Path="/5E686310" Ref="#PWR?"  Part="1"
-F 0 "#PWR023" H 4900 3100 50  0001 C CNN
+F 0 "#PWR09" H 4900 3100 50  0001 C CNN
 F 1 "+2V8" V 4915 3378 50  0000 L CNN
 F 2 "" H 4900 3250 50  0001 C CNN

Commit message: removed psi-things pins, added transceiver MCP2551 for CAN, changed motors input protocol, RS must be chosen 1 or 10 kohms, and a foot print for a potentitial 120 ohms resistor is present for CAN bus end.
Changed lines of the file:
@@
 $Descr A4 11693 8268
 encoding utf-8
-Sheet 3 24
+Sheet 3 23
 Title ""
 Date ""
@@
 AR Path="/5E68B664/5E684EEF" Ref="J9"  Part="1"
 AR Path="/5E68B669/5E684EEF" Ref="J10"  Part="1"
-F 0 "J3" H 5330 3492 50  0000 L CNN
+F 0 "J10" H 5330 3492 50  0000 L CNN
 F 1 "ToF" H 5330 3401 50  0000 L CNN
 F 2 "Connector_JST:JST_PH_B5B-PH-K_1x05_P2.00mm_Vertical" H 5250 3450 50  0001 C CNN
@@
 $EndComp
 $Comp
-L shield_etage2-rescue:GND-power-shield_etage2-rescue #PWR010
+L shield_etage2-rescue:GND-power-shield_etage2-rescue #PWR09
 U 1 1 5E6859B3
 P 4900 3650
-AR Path="/5E678883/5E6859B3" Ref="#PWR010"  Part="1"
-AR Path="/5E688559/5E6859B3" Ref="#PWR012"  Part="1"
-AR Path="/5E688F3B/5E6859B3" Ref="#PWR014"  Part="1"
-AR Path="/5E689251/5E6859B3" Ref="#PWR016"  Part="1"
-AR Path="/5E68B65A/5E6859B3" Ref="#PWR018"  Part="1"
-AR Path="/5E68B65F/5E6859B3" Ref="#PWR020"  Part="1"
-AR Path="/5E68B664/5E6859B3" Ref="#PWR022"  Part="1"
-AR Path="/5E68B669/5E6859B3" Ref="#PWR024"  Part="1"
-F 0 "#PWR010" H 4900 3400 50  0001 C CNN
+AR Path="/5E678883/5E6859B3" Ref="#PWR09"  Part="1"
+AR Path="/5E688559/5E6859B3" Ref="#PWR011"  Part="1"
+AR Path="/5E688F3B/5E6859B3" Ref="#PWR013"  Part="1"
+AR Path="/5E689251/5E6859B3" Ref="#PWR015"  Part="1"
+AR Path="/5E68B65A/5E6859B3" Ref="#PWR017"  Part="1"
+AR Path="/5E68B65F/5E6859B3" Ref="#PWR019"  Part="1"
+AR Path="/5E68B664/5E6859B3" Ref="#PWR021"  Part="1"
+AR Path="/5E68B669/5E6859B3" Ref="#PWR023"  Part="1"
+F 0 "#PWR023" H 4900 3400 50  0001 C CNN
 F 1 "GND" V 4905 3522 50  0000 R CNN
 F 2 "" H 4900 3650 50  0001 C CNN
@@
 $EndComp
 $Comp
-L shield_etage2-rescue:+2V8-power-shield_etage2-rescue #PWR09
+L shield_etage2-rescue:+2V8-power-shield_etage2-rescue #PWR08
 U 1 1 5E686310
 P 4900 3250
-AR Path="/5E678883/5E686310" Ref="#PWR09"  Part="1"
-AR Path="/5E688559/5E686310" Ref="#PWR011"  Part="1"
-AR Path="/5E688F3B/5E686310" Ref="#PWR013"  Part="1"
-AR Path="/5E689251/5E686310" Ref="#PWR015"  Part="1"
-AR Path="/5E68B65A/5E686310" Ref="#PWR017"  Part="1"
-AR Path="/5E68B65F/5E686310" Ref="#PWR019"  Part="1"
-AR Path="/5E68B664/5E686310" Ref="#PWR021"  Part="1"
-AR Path="/5E68B669/5E686310" Ref="#PWR023"  Part="1"
+AR Path="/5E678883/5E686310" Ref="#PWR08"  Part="1"
+AR Path="/5E688559/5E686310" Ref="#PWR010"  Part="1"
+AR Path="/5E688F3B/5E686310" Ref="#PWR012"  Part="1"
+AR Path="/5E689251/5E686310" Ref="#PWR014"  Part="1"
+AR Path="/5E68B65A/5E686310" Ref="#PWR016"  Part="1"
+AR Path="/5E68B65F/5E686310" Ref="#PWR018"  Part="1"
+AR Path="/5E68B664/5E686310" Ref="#PWR020"  Part="1"
+AR Path="/5E68B669/5E686310" Ref="#PWR022"  Part="1"
 AR Path="/5E686310" Ref="#PWR?"  Part="1"
-F 0 "#PWR09" H 4900 3100 50  0001 C CNN
+F 0 "#PWR022" H 4900 3100 50  0001 C CNN
 F 1 "+2V8" V 4915 3378 50  0000 L CNN
 F 2 "" H 4900 3250 50  0001 C CNN

Commit message: correction mm -> inch, empreinte du bouton
Parts:
- J3: footprint Connector_JST:JST_PH_B5B-PH-K_1x05_P2.00mm_Vertical -> Connector_JST:JST_XH_B5B-XH-A_1x05_P2.50mm_Vertical
Changed lines of the file:
@@
 $Descr A4 11693 8268
 encoding utf-8
-Sheet 3 23
+Sheet 9 23
 Title ""
 Date ""
@@
 AR Path="/5E68B664/5E684EEF" Ref="J9"  Part="1"
 AR Path="/5E68B669/5E684EEF" Ref="J10"  Part="1"
-F 0 "J10" H 5330 3492 50  0000 L CNN
+F 0 "J9" H 5330 3492 50  0000 L CNN
 F 1 "ToF" H 5330 3401 50  0000 L CNN
-F 2 "Connector_JST:JST_PH_B5B-PH-K_1x05_P2.00mm_Vertical" H 5250 3450 50  0001 C CNN
+F 2 "Connector_JST:JST_XH_B5B-XH-A_1x05_P2.50mm_Vertical" H 5250 3450 50  0001 C CNN
 F 3 "~" H 5250 3450 50  0001 C CNN
 	1    5250 3450
