File: Driver_moteurs.sch (KiCad schematic (older format))
At the start: 9 parts, among them U5 L293D

Commit message: Add files via upload
Parts:
- added C13, C14: 100n, symbol Device:C
- gave numbers to parts that had none: 8
Connections:
- net +5V: now also C13.2
- net GND: now also C13.1, C14.1
- net at R15.1, U2.1 (ADJ), U5.8 (VCC2): now also C14.2
Changed lines of the file:
@@
 $Descr A4 11693 8268
 encoding utf-8
-Sheet 16 23
+Sheet 16 22
 Title ""
 Date ""
@@
 AR Path="/5E62FD4D/5E80BDFA" Ref="R?"  Part="1"
 AR Path="/5E66627C/5E80BDFA" Ref="R?"  Part="1"
-AR Path="/5E6AC71D/5E80BDFA" Ref="R?"  Part="1"
-F 0 "R?" H 2470 4346 50  0000 L CNN
+AR Path="/5E6AC71D/5E80BDFA" Ref="R11"  Part="1"
+F 0 "R11" H 2470 4346 50  0000 L CNN
 F 1 "Pull" H 2470 4255 50  0000 L CNN
 F 2 "" V 2330 4300 50  0001 C CNN
@@
 AR Path="/5E62FD4D/5E80BE00" Ref="R?"  Part="1"
 AR Path="/5E66627C/5E80BE00" Ref="R?"  Part="1"
-AR Path="/5E6AC71D/5E80BE00" Ref="R?"  Part="1"
-F 0 "R?" H 3170 4346 50  0000 L CNN
+AR Path="/5E6AC71D/5E80BE00" Ref="R13"  Part="1"
+F 0 "R13" H 3170 4346 50  0000 L CNN
 F 1 "Pull" H 3170 4255 50  0000 L CNN
 F 2 "" V 3030 4300 50  0001 C CNN
@@
 AR Path="/5E62FD4D/5E80BE08" Ref="Q?"  Part="1"
 AR Path="/5E66627C/5E80BE08" Ref="Q?"  Part="1"
-AR Path="/5E6AC71D/5E80BE08" Ref="Q?"  Part="1"
-F 0 "Q?" V 3001 4450 50  0000 C CNN
+AR Path="/5E6AC71D/5E80BE08" Ref="Q5"  Part="1"
+F 0 "Q5" V 3001 4450 50  0000 C CNN
 F 1 "BSS138" V 3092 4450 50  0000 C CNN
 F 2 "Package_TO_SOT_SMD:SOT-23" H 2950 4375 50  0001 L CIN
@@
 L power:+3V3 #PWR?
 U 1 1 5E80BE1C
-P 2400 4050
+P 2400 4000
 AR Path="/5E66627C/5E80BE1C" Ref="#PWR?"  Part="1"
-AR Path="/5E6AC71D/5E80BE1C" Ref="#PWR?"  Part="1"
-F 0 "#PWR?" H 2400 3900 50  0001 C CNN
-F 1 "+3V3" H 2415 4223 50  0000 C CNN
-F 2 "" H 2400 4050 50  0001 C CNN
-F 3 "" H 2400 4050 50  0001 C CNN
-	1    2400 4050
+AR Path="/5E6AC71D/5E80BE1C" Ref="#PWR0109"  Part="1"
+F 0 "#PWR0109" H 2400 3850 50  0001 C CNN
+F 1 "+3V3" H 2415 4173 50  0000 C CNN
+F 2 "" H 2400 4000 50  0001 C CNN
+F 3 "" H 2400 4000 50  0001 C CNN
+	1    2400 4000
 	1    0    0    -1
 $EndComp
@@
 	2400 4550 2100 4550
 Connection ~ 2400 4550
-Connection ~ 2400 4050
-$Comp
-L power:+5V #PWR?
+$Comp
+L power:+5V #PWR0110
 U 1 1 5E8288E7
 P 3100 4050
-F 0 "#PWR?" H 3100 3900 50  0001 C CNN
+F 0 "#PWR0110" H 3100 3900 50  0001 C CNN
 F 1 "+5V" H 3115 4223 50  0000 C CNN
 F 2 "" H 3100 4050 50  0001 C CNN
@@
 AR Path="/5E62FD4D/5E8639E8" Ref="R?"  Part="1"
 AR Path="/5E66627C/5E8639E8" Ref="R?"  Part="1"
-AR Path="/5E6AC71D/5E8639E8" Ref="R?"  Part="1"
-F 0 "R?" H 2470 5596 50  0000 L CNN
+AR Path="/5E6AC71D/5E8639E8" Ref="R12"  Part="1"
+F 0 "R12" H 2470 5596 50  0000 L CNN
 F 1 "Pull" H 2470 5505 50  0000 L CNN
 F 2 "" V 2330 5550 50  0001 C CNN
@@
 AR Path="/5E62FD4D/5E8639EE" Ref="R?"  Part="1"
 AR Path="/5E66627C/5E8639EE" Ref="R?"  Part="1"
-AR Path="/5E6AC71D/5E8639EE" Ref="R?"  Part="1"
-F 0 "R?" H 3170 5596 50  0000 L CNN
+AR Path="/5E6AC71D/5E8639EE" Ref="R14"  Part="1"
+F 0 "R14" H 3170 5596 50  0000 L CNN
 F 1 "Pull" H 3170 5505 50  0000 L CNN
 F 2 "" V 3030 5550 50  0001 C CNN
@@
 AR Path="/5E62FD4D/5E8639F4" Ref="Q?"  Part="1"
 AR Path="/5E66627C/5E8639F4" Ref="Q?"  Part="1"
-AR Path="/5E6AC71D/5E8639F4" Ref="Q?"  Part="1"
-F 0 "Q?" V 3001 5700 50  0000 C CNN
+AR Path="/5E6AC71D/5E8639F4" Ref="Q6"  Part="1"
+F 0 "Q6" V 3001 5700 50  0000 C CNN
 F 1 "BSS138" V 3092 5700 50  0000 C CNN
 F 2 "Package_TO_SOT_SMD:SOT-23" H 2950 5625 50  0001 L CIN
@@
 L power:+3V3 #PWR?
 U 1 1 5E8639FB
-P 2400 5300
+P 2400 5250
 AR Path="/5E66627C/5E8639FB" Ref="#PWR?"  Part="1"
-AR Path="/5E6AC71D/5E8639FB" Ref="#PWR?"  Part="1"
-F 0 "#PWR?" H 2400 5150 50  0001 C CNN
-F 1 "+3V3" H 2415 5473 50  0000 C CNN
-F 2 "" H 2400 5300 50  0001 C CNN
-F 3 "" H 2400 5300 50  0001 C CNN
-	1    2400 5300
+AR Path="/5E6AC71D/5E8639FB" Ref="#PWR0111"  Part="1"
+F 0 "#PWR0111" H 2400 5100 50  0001 C CNN
+F 1 "+3V3" H 2415 5423 50  0000 C CNN
+F 2 "" H 2400 5250 50  0001 C CNN
+F 3 "" H 2400 5250 50  0001 C CNN
+	1    2400 5250
 	1    0    0    -1
 $EndComp
@@
 	2400 5800 2100 5800
 Connection ~ 2400 5800
-Connection ~ 2400 5300
-$Comp
-L power:+5V #PWR?
+$Comp
+L power:+5V #PWR0112
 U 1 1 5E863A0A
 P 3100 5300
-F 0 "#PWR?" H 3100 5150 50  0001 C CNN
+F 0 "#PWR0112" H 3100 5150 50  0001 C CNN
 F 1 "+5V" H 3115 5473 50  0000 C CNN
 F 2 "" H 3100 5300 50  0001 C CNN
@@
 pwm_drapeau_enable
 $Comp
-L power:+5V #PWR?
+L power:+5V #PWR0113
 U 1 1 5E8690D7
 P 6000 3400
-F 0 "#PWR?" H 6000 3250 50  0001 C CNN
+F 0 "#PWR0113" H 6000 3250 50  0001 C CNN
 F 1 "+5V" H 6015 3573 50  0000 C CNN
 F 2 "" H 6000 3400 50  0001 C CNN
@@
 	1    0    0    -1
 $EndComp
-Wire Wire Line
-	6000 3400 6000 3750
 Text Notes 3950 1300 0    50   ~ 0
 FCL = Fault Current Limiter\nPour éviter un pic de courant si\nun moteur grille
@@
 AR Path="/5E686EE6/5E7F198B" Ref="U?"  Part="1"
 AR Path="/5E6883CB/5E7F198B" Ref="U?"  Part="1"
-AR Path="/5E6AC71D/5E7F198B" Ref="U?"  Part="1"
-F 0 "U?" H 4400 1992 50  0000 C CNN
+AR Path="/5E6AC71D/5E7F198B" Ref="U2"  Part="1"
+F 0 "U2" H 4400 1992 50  0000 C CNN
 F 1 "LM317_TO3" H 4400 1901 50  0000 C CNN
 F 2 "Package_TO_SOT_THT:TO-3" H 4400 1950 50  0001 C CIN
@@
 AR Path="/5E686EE6/5E7F1992" Ref="R?"  Part="1"
 AR Path="/5E6883CB/5E7F1992" Ref="R?"  Part="1"
-AR Path="/5E6AC71D/5E7F1992" Ref="R?"  Part="1"
-F 0 "R?" V 4743 1750 50  0000 C CNN
+AR Path="/5E6AC71D/5E7F1992" Ref="R15"  Part="1"
+F 0 "R15" V 4743 1750 50  0000 C CNN
 F 1 "R" V 4834 1750 50  0000 C CNN
 F 2 "" V 4880 1750 50  0001 C CNN
@@
 Pour le contrôle des moteurs :\nMoteur 1 en sens direct : \n- bras_sens_direct = HIGH\n- bras_sens_inverse = LOW\nMoteur 1 en sens inverse : \n- bras_sens_direct = LOW\n- bras_sens_inverse = HIGH\n\nsimilairement pour le moteur du drapeau\n\nLa vitesse est contrôlée en modulant via PWM \nl'entrée "ENABLE" du pont en H
 Wire Wire Line
-	6200 1750 6200 3750
-Wire Wire Line
 	5150 1750 6200 1750
+$Comp
+L Device:C C?
+U 1 1 5E83530F
+P 5850 3500
+AR Path="/5E627338/5E83530F" Ref="C?"  Part="1"
+AR Path="/5E6AC71D/5E83530F" Ref="C13"  Part="1"
+F 0 "C13" V 5598 3500 50  0000 C CNN
+F 1 "100n" V 5689 3500 50  0000 C CNN
+F 2 "" H 5888 3350 50  0001 C CNN
+F 3 "~" H 5850 3500 50  0001 C CNN
+	1    5850 3500
+	0    -1   -1   0
+$EndComp
+$Comp
+L power:GND #PWR?
+U 1 1 5E835315
+P 5700 3500
+AR Path="/5E627338/5E835315" Ref="#PWR?"  Part="1"
+AR Path="/5E6AC71D/5E835315" Ref="#PWR0129"  Part="1"
+F 0 "#PWR0129" H 5700 3250 50  0001 C CNN
+F 1 "GND" V 5705 3372 50  0000 R CNN
+F 2 "" H 5700 3500 50  0001 C CNN
+F 3 "" H 5700 3500 50  0001 C CNN
+	1    5700 3500
+	0    1    1    0
+$EndComp
+$Comp
+L Device:C C?
+U 1 1 5E8363F0
+P 6350 3500
+AR Path="/5E627338/5E8363F0" Ref="C?"  Part="1"
+AR Path="/5E6AC71D/5E8363F0" Ref="C14"  Part="1"
+F 0 "C14" V 6098 3500 50  0000 C CNN
+F 1 "100n" V 6189 3500 50  0000 C CNN
+F 2 "" H 6388 3350 50  0001 C CNN
+F 3 "~" H 6350 3500 50  0001 C CNN
+	1    6350 3500
+	0    1    1    0
+$EndComp
+$Comp
+L power:GND #PWR?
+U 1 1 5E8363F6
+P 6500 3500
+AR Path="/5E627338/5E8363F6" Ref="#PWR?"  Part="1"
+AR Path="/5E6AC71D/5E8363F6" Ref="#PWR0130"  Part="1"
+F 0 "#PWR0130" H 6500 3250 50  0001 C CNN
+F 1 "GND" V 6505 3372 50  0000 R CNN
+F 2 "" H 6500 3500 50  0001 C CNN
+F 3 "" H 6500 3500 50  0001 C CNN
+	1    6500 3500
+	0    -1   -1   0
+$EndComp
+Wire Wire Line
+	6000 3400 6000 3500
+Wire Wire Line
+	6200 1750 6200 3500
+Wire Wire Line
+	6200 3500 6200 3750
+Connection ~ 6200 3500
+Wire Wire Line
+	6000 3500 6000 3750
+Connection ~ 6000 3500
+Wire Wire Line
+	2400 5300 2400 5250
+Connection ~ 2400 5300
+Wire Wire Line
+	2400 4000 2400 4050
+Connection ~ 2400 4050
+$Comp
+L power:PWR_FLAG #FLG0101
+U 1 1 5E94CE45
+P 6200 1750
+F 0 "#FLG0101" H 6200 1825 50  0001 C CNN
+F 1 "PWR_FLAG" H 6200 1923 50  0000 C CNN
+F 2 "" H 6200 1750 50  0001 C CNN
+F 3 "~" H 6200 1750 50  0001 C CNN
+	1    6200 1750
+	1    0    0    -1
+$EndComp
+Connection ~ 6200 1750
 $EndSCHEMATC

Commit message: Add files via upload
Parts:
- C13, C14: footprint (none) -> Capacitor_SMD:C_0805_2012Metric_Pad1.15x1.40mm_HandSolder
- R11, R12, R13, R14: footprint (none) -> Resistor_SMD:R_0805_2012Metric_Pad1.15x1.40mm_HandSolder
- R15: value R -> 1.2; footprint (none) -> Resistor_THT:R_Axial_DIN0414_L11.9mm_D4.5mm_P15.24mm_Horizontal
- U2: footprint Package_TO_SOT_THT:TO-3 -> Package_TO_SOT_THT:TO-220-3_Vertical
Changed lines of the file:
@@
 EESchema Schematic File Version 4
-LIBS:kicad_master-cache
 EELAYER 30 0
 EELAYER END
 $Descr A4 11693 8268
 encoding utf-8
-Sheet 16 22
+Sheet 16 21
 Title ""
 Date ""
@@
 F 0 "R11" H 2470 4346 50  0000 L CNN
 F 1 "Pull" H 2470 4255 50  0000 L CNN
-F 2 "" V 2330 4300 50  0001 C CNN
+F 2 "Resistor_SMD:R_0805_2012Metric_Pad1.15x1.40mm_HandSolder" V 2330 4300 50  0001 C CNN
 F 3 "~" H 2400 4300 50  0001 C CNN
 	1    2400 4300
@@
 F 0 "R13" H 3170 4346 50  0000 L CNN
 F 1 "Pull" H 3170 4255 50  0000 L CNN
-F 2 "" V 3030 4300 50  0001 C CNN
+F 2 "Resistor_SMD:R_0805_2012Metric_Pad1.15x1.40mm_HandSolder" V 3030 4300 50  0001 C CNN
 F 3 "~" H 3100 4300 50  0001 C CNN
 	1    3100 4300
@@
 F 0 "R12" H 2470 5596 50  0000 L CNN
 F 1 "Pull" H 2470 5505 50  0000 L CNN
-F 2 "" V 2330 5550 50  0001 C CNN
+F 2 "Resistor_SMD:R_0805_2012Metric_Pad1.15x1.40mm_HandSolder" V 2330 5550 50  0001 C CNN
 F 3 "~" H 2400 5550 50  0001 C CNN
 	1    2400 5550
@@
 F 0 "R14" H 3170 5596 50  0000 L CNN
 F 1 "Pull" H 3170 5505 50  0000 L CNN
-F 2 "" V 3030 5550 50  0001 C CNN
+F 2 "Resistor_SMD:R_0805_2012Metric_Pad1.15x1.40mm_HandSolder" V 3030 5550 50  0001 C CNN
 F 3 "~" H 3100 5550 50  0001 C CNN
 	1    3100 5550
@@
 F 0 "U2" H 4400 1992 50  0000 C CNN
 F 1 "LM317_TO3" H 4400 1901 50  0000 C CNN
-F 2 "Package_TO_SOT_THT:TO-3" H 4400 1950 50  0001 C CIN
+F 2 "Package_TO_SOT_THT:TO-220-3_Vertical" H 4400 1950 50  0001 C CIN
 F 3 "http://www.ti.com/lit/ds/symlink/lm317.pdf" H 4400 1750 50  0001 C CNN
 	1    4400 1750
@@
 AR Path="/5E6AC71D/5E7F1992" Ref="R15"  Part="1"
 F 0 "R15" V 4743 1750 50  0000 C CNN
-F 1 "R" V 4834 1750 50  0000 C CNN
-F 2 "" V 4880 1750 50  0001 C CNN
+F 1 "1.2" V 4834 1750 50  0000 C CNN
+F 2 "Resistor_THT:R_Axial_DIN0414_L11.9mm_D4.5mm_P15.24mm_Horizontal" V 4880 1750 50  0001 C CNN
 F 3 "~" H 4950 1750 50  0001 C CNN
 	1    4950 1750
@@
 F 0 "C13" V 5598 3500 50  0000 C CNN
 F 1 "100n" V 5689 3500 50  0000 C CNN
-F 2 "" H 5888 3350 50  0001 C CNN
+F 2 "Capacitor_SMD:C_0805_2012Metric_Pad1.15x1.40mm_HandSolder" H 5888 3350 50  0001 C CNN
 F 3 "~" H 5850 3500 50  0001 C CNN
 	1    5850 3500
@@
 F 0 "C14" V 6098 3500 50  0000 C CNN
 F 1 "100n" V 6189 3500 50  0000 C CNN
-F 2 "" H 6388 3350 50  0001 C CNN
+F 2 "Capacitor_SMD:C_0805_2012Metric_Pad1.15x1.40mm_HandSolder" H 6388 3350 50  0001 C CNN
 F 3 "~" H 6350 3500 50  0001 C CNN
 	1    6350 3500

Commit message: avancement général du routage
Parts:
- C13, C14: symbol Device:C -> shield_etage2-rescue:C-Device
- Q5, Q6: symbol Transistor_FET:BSS138 -> shield_etage2-rescue:BSS138-Transistor_FET
- R11, R12, R13, R14, R15: symbol Device:R -> shield_etage2-rescue:R-Device
- U2: symbol Regulator_Linear:LM317_TO3 -> shield_etage2-rescue:LM317_TO3-Regulator_Linear
- U5: symbol Driver_Motor:L293D -> shield_etage2-rescue:L293D-Driver_Motor
Changed lines of the file:
@@
 $EndDescr
 $Comp
-L Driver_Motor:L293D U5
+L shield_etage2-rescue:L293D-Driver_Motor U5
 U 1 1 5E6ACB12
 P 6100 4750
@@
 Connection ~ 6000 5750
 $Comp
-L power:GND #PWR0107
+L shield_etage2-rescue:GND-power #PWR0107
 U 1 1 5E6AEBFC
 P 6000 5900
@@
 moteur2_pin1
 $Comp
-L Device:R R?
+L shield_etage2-rescue:R-Device R?
 U 1 1 5E80BDFA
 P 2400 4300
@@
 $EndComp
 $Comp
-L Device:R R?
+L shield_etage2-rescue:R-Device R?
 U 1 1 5E80BE00
 P 3100 4300
@@
 $EndComp
 $Comp
-L Transistor_FET:BSS138 Q?
+L shield_etage2-rescue:BSS138-Transistor_FET Q?
 U 1 1 5E80BE08
 P 2750 4450
@@
 	2950 4550 3100 4550
 $Comp
-L power:+3V3 #PWR?
+L shield_etage2-rescue:+3V3-power #PWR?
 U 1 1 5E80BE1C
 P 2400 4000
@@
 Connection ~ 2400 4550
 $Comp
-L power:+5V #PWR0110
+L shield_etage2-rescue:+5V-power #PWR0110
 U 1 1 5E8288E7
 P 3100 4050
@@
 	3100 4050 3100 4150
 $Comp
-L Device:R R?
+L shield_etage2-rescue:R-Device R?
 U 1 1 5E8639E8
 P 2400 5550
@@
 $EndComp
 $Comp
-L Device:R R?
+L shield_etage2-rescue:R-Device R?
 U 1 1 5E8639EE
 P 3100 5550
@@
 $EndComp
 $Comp
-L Transistor_FET:BSS138 Q?
+L shield_etage2-rescue:BSS138-Transistor_FET Q?
 U 1 1 5E8639F4
 P 2750 5700
@@
 	2950 5800 3100 5800
 $Comp
-L power:+3V3 #PWR?
+L shield_etage2-rescue:+3V3-power #PWR?
 U 1 1 5E8639FB
 P 2400 5250
@@
 Connection ~ 2400 5800
 $Comp
-L power:+5V #PWR0112
+L shield_etage2-rescue:+5V-power #PWR0112
 U 1 1 5E863A0A
 P 3100 5300
@@
 pwm_drapeau_enable
 $Comp
-L power:+5V #PWR0113
+L shield_etage2-rescue:+5V-power #PWR0113
 U 1 1 5E8690D7
 P 6000 3400
@@
 FCL = Fault Current Limiter\nPour éviter un pic de courant si\nun moteur grille
 $Comp
-L Regulator_Linear:LM317_TO3 U?
+L shield_etage2-rescue:LM317_TO3-Regulator_Linear U?
 U 1 1 5E7F198B
 P 4400 1750
@@
 Is = 1.25/R\n
 $Comp
-L Device:R R?
+L shield_etage2-rescue:R-Device R?
 U 1 1 5E7F1992
 P 4950 1750
@@
 	5150 1750 6200 1750
 $Comp
-L Device:C C?
+L shield_etage2-rescue:C-Device C?
 U 1 1 5E83530F
 P 5850 3500
@@
 $EndComp
 $Comp
-L power:GND #PWR?
+L shield_etage2-rescue:GND-power #PWR?
 U 1 1 5E835315
 P 5700 3500
@@
 $EndComp
 $Comp
-L Device:C C?
+L shield_etage2-rescue:C-Device C?
 U 1 1 5E8363F0
 P 6350 3500
@@
 $EndComp
 $Comp
-L power:GND #PWR?
+L shield_etage2-rescue:GND-power #PWR?
 U 1 1 5E8363F6
 P 6500 3500
@@
 Connection ~ 2400 4050
 $Comp
-L power:PWR_FLAG #FLG0101
+L shield_etage2-rescue:PWR_FLAG-power #FLG0101
 U 1 1 5E94CE45
 P 6200 1750
