File: FinDeCourse.sch (KiCad schematic (older format))
At the start: 2 parts, among them J13 Conn_01x02

Commit message: Add files via upload
Parts:
- removed R12: 10k, symbol Device:R
- added C6: 100n, symbol Device:C
Connections:
- net GND: now also C6.2
- net STM32_GPIO: now also C6.1
Other:
- moved on the sheet: J13
Changed lines of the file:
@@
 $Descr A4 11693 8268
 encoding utf-8
-Sheet 19 23
+Sheet 19 22
 Title ""
 Date ""
@@
 STM32_GPIO
 $Comp
-L Device:R R12
-U 1 1 5E7DB152
-P 6800 2250
-AR Path="/5E6942FF/5E7DB152" Ref="R12"  Part="1"
-AR Path="/5E69459B/5E7DB152" Ref="R13"  Part="1"
-F 0 "R12" H 6870 2296 50  0000 L CNN
-F 1 "10k" H 6870 2205 50  0000 L CNN
-F 2 "" V 6730 2250 50  0001 C CNN
-F 3 "~" H 6800 2250 50  0001 C CNN
-	1    6800 2250
+L Connector_Generic:Conn_01x02 J13
+U 1 1 5E7DC2F9
+P 7350 2600
+AR Path="/5E6942FF/5E7DC2F9" Ref="J13"  Part="1"
+AR Path="/5E69459B/5E7DC2F9" Ref="J14"  Part="1"
+F 0 "J13" H 7268 2275 50  0000 C CNN
+F 1 "Conn_01x02" H 7268 2366 50  0000 C CNN
+F 2 "" H 7350 2600 50  0001 C CNN
+F 3 "~" H 7350 2600 50  0001 C CNN
+	1    7350 2600
 	1    0    0    -1
 $EndComp
 $Comp
-L power:+5V #PWR0103
-U 1 1 5E7DB84D
-P 6800 1950
-AR Path="/5E6942FF/5E7DB84D" Ref="#PWR0103"  Part="1"
-AR Path="/5E69459B/5E7DB84D" Ref="#PWR0105"  Part="1"
-F 0 "#PWR0103" H 6800 1800 50  0001 C CNN
-F 1 "+5V" H 6815 2123 50  0000 C CNN
-F 2 "" H 6800 1950 50  0001 C CNN
-F 3 "" H 6800 1950 50  0001 C CNN
-	1    6800 1950
+L power:GND #PWR0104
+U 1 1 5E7E6F28
+P 6450 2900
+AR Path="/5E6942FF/5E7E6F28" Ref="#PWR0104"  Part="1"
+AR Path="/5E69459B/5E7E6F28" Ref="#PWR0106"  Part="1"
+F 0 "#PWR0104" H 6450 2650 50  0001 C CNN
+F 1 "GND" H 6455 2727 50  0000 C CNN
+F 2 "" H 6450 2900 50  0001 C CNN
+F 3 "" H 6450 2900 50  0001 C CNN
+	1    6450 2900
 	1    0    0    -1
 $EndComp
+Text Notes 7450 2500 0    50   ~ 0
+Les capteurs de fin de course permettent de savoir si le moteur bras \net le moteur drapeau sont arrivés au bout de leur ouverture, et éviter\n de continuer à commander les moteurs en forçant
 $Comp
-L Connector_Generic:Conn_01x02 J13
-U 1 1 5E7DC2F9
-P 7350 3000
-AR Path="/5E6942FF/5E7DC2F9" Ref="J13"  Part="1"
-AR Path="/5E69459B/5E7DC2F9" Ref="J14"  Part="1"
-F 0 "J13" H 7268 2675 50  0000 C CNN
-F 1 "Conn_01x02" H 7268 2766 50  0000 C CNN
-F 2 "" H 7350 3000 50  0001 C CNN
-F 3 "~" H 7350 3000 50  0001 C CNN
-	1    7350 3000
+L Device:C C6
+U 1 1 5E835C66
+P 6450 2750
+AR Path="/5E69459B/5E835C66" Ref="C6"  Part="1"
+AR Path="/5E6942FF/5E835C66" Ref="C7"  Part="1"
+F 0 "C7" H 6565 2796 50  0000 L CNN
+F 1 "100n" H 6565 2705 50  0000 L CNN
+F 2 "" H 6488 2600 50  0001 C CNN
+F 3 "~" H 6450 2750 50  0001 C CNN
+	1    6450 2750
+	1    0    0    -1
+$EndComp
+Connection ~ 6450 2600
+Wire Wire Line
+	6450 2600 6150 2600
+Wire Wire Line
+	6450 2600 7150 2600
+$Comp
+L power:GND #PWR0118
+U 1 1 5E8388AC
+P 6850 2900
+AR Path="/5E6942FF/5E8388AC" Ref="#PWR0118"  Part="1"
+AR Path="/5E69459B/5E8388AC" Ref="#PWR0117"  Part="1"
+F 0 "#PWR0118" H 6850 2650 50  0001 C CNN
+F 1 "GND" H 6855 2727 50  0000 C CNN
+F 2 "" H 6850 2900 50  0001 C CNN
+F 3 "" H 6850 2900 50  0001 C CNN
+	1    6850 2900
 	1    0    0    -1
 $EndComp
 Wire Wire Line
-	6800 2600 6800 2400
+	6850 2900 6850 2700
 Wire Wire Line
-	6800 2100 6800 1950
-Wire Wire Line
-	6800 2600 6150 2600
-Wire Wire Line
-	6800 2600 6800 3000
-Connection ~ 6800 2600
-$Comp
-L power:GND #PWR0104
-U 1 1 5E7E6F28
-P 6800 3350
-AR Path="/5E6942FF/5E7E6F28" Ref="#PWR0104"  Part="1"
-AR Path="/5E69459B/5E7E6F28" Ref="#PWR0106"  Part="1"
-F 0 "#PWR0104" H 6800 3100 50  0001 C CNN
-F 1 "GND" H 6805 3177 50  0000 C CNN
-F 2 "" H 6800 3350 50  0001 C CNN
-F 3 "" H 6800 3350 50  0001 C CNN
-	1    6800 3350
-	1    0    0    -1
-$EndComp
-Wire Wire Line
-	7150 3100 6800 3100
-Wire Wire Line
-	6800 3100 6800 3350
-Wire Wire Line
-	6800 3000 7150 3000
-Text Notes 7450 2500 0    50   ~ 0
-Les capteurs de fin de course permettent de savoir si le moteur bras \net le moteur drapeau sont arrivés au bout de leur ouverture, et éviter\n de continuer à commander les moteurs en forçant
+	6850 2700 7150 2700
 $EndSCHEMATC

Commit message: Add files via upload
Parts:
- C6: footprint (none) -> Capacitor_SMD:C_0805_2012Metric_Pad1.15x1.40mm_HandSolder
- J13: value Conn_01x02 -> butee; footprint (none) -> Connector_JST:JST_PH_B2B-PH-K_1x02_P2.00mm_Vertical
Changed lines of the file:
@@
 EESchema Schematic File Version 4
-LIBS:kicad_master-cache
 EELAYER 30 0
 EELAYER END
 $Descr A4 11693 8268
 encoding utf-8
-Sheet 19 22
+Sheet 17 21
 Title ""
 Date ""
@@
 AR Path="/5E6942FF/5E7DC2F9" Ref="J13"  Part="1"
 AR Path="/5E69459B/5E7DC2F9" Ref="J14"  Part="1"
-F 0 "J13" H 7268 2275 50  0000 C CNN
-F 1 "Conn_01x02" H 7268 2366 50  0000 C CNN
-F 2 "" H 7350 2600 50  0001 C CNN
+F 0 "J14" H 7268 2275 50  0000 C CNN
+F 1 "butee" H 7268 2366 50  0000 C CNN
+F 2 "Connector_JST:JST_PH_B2B-PH-K_1x02_P2.00mm_Vertical" H 7350 2600 50  0001 C CNN
 F 3 "~" H 7350 2600 50  0001 C CNN
 	1    7350 2600
@@
 AR Path="/5E69459B/5E835C66" Ref="C6"  Part="1"
 AR Path="/5E6942FF/5E835C66" Ref="C7"  Part="1"
-F 0 "C7" H 6565 2796 50  0000 L CNN
+F 0 "C6" H 6565 2796 50  0000 L CNN
 F 1 "100n" H 6565 2705 50  0000 L CNN
-F 2 "" H 6488 2600 50  0001 C CNN
+F 2 "Capacitor_SMD:C_0805_2012Metric_Pad1.15x1.40mm_HandSolder" H 6488 2600 50  0001 C CNN
 F 3 "~" H 6450 2750 50  0001 C CNN
 	1    6450 2750

Commit message: avancement général du routage
Parts:
- C6: symbol Device:C -> shield_etage2-rescue:C-Device
- J13: symbol Connector_Generic:Conn_01x02 -> shield_etage2-rescue:Conn_01x02-Connector_Generic
Changed lines of the file:
@@
 STM32_GPIO
 $Comp
-L Connector_Generic:Conn_01x02 J13
+L shield_etage2-rescue:Conn_01x02-Connector_Generic J13
 U 1 1 5E7DC2F9
 P 7350 2600
@@
 $EndComp
 $Comp
-L power:GND #PWR0104
+L shield_etage2-rescue:GND-power #PWR0104
 U 1 1 5E7E6F28
 P 6450 2900
 AR Path="/5E6942FF/5E7E6F28" Ref="#PWR0104"  Part="1"
 AR Path="/5E69459B/5E7E6F28" Ref="#PWR0106"  Part="1"
-F 0 "#PWR0104" H 6450 2650 50  0001 C CNN
+F 0 "#PWR0106" H 6450 2650 50  0001 C CNN
 F 1 "GND" H 6455 2727 50  0000 C CNN
 F 2 "" H 6450 2900 50  0001 C CNN
@@
 Les capteurs de fin de course permettent de savoir si le moteur bras \net le moteur drapeau sont arrivés au bout de leur ouverture, et éviter\n de continuer à commander les moteurs en forçant
 $Comp
-L Device:C C6
+L shield_etage2-rescue:C-Device C6
 U 1 1 5E835C66
 P 6450 2750
@@
 	6450 2600 7150 2600
 $Comp
-L power:GND #PWR0118
+L shield_etage2-rescue:GND-power #PWR0118
 U 1 1 5E8388AC
 P 6850 2900
 AR Path="/5E6942FF/5E8388AC" Ref="#PWR0118"  Part="1"
 AR Path="/5E69459B/5E8388AC" Ref="#PWR0117"  Part="1"
-F 0 "#PWR0118" H 6850 2650 50  0001 C CNN
+F 0 "#PWR0117" H 6850 2650 50  0001 C CNN
 F 1 "GND" H 6855 2727 50  0000 C CNN
 F 2 "" H 6850 2900 50  0001 C CNN
