File: LevelShifter_ShiftRegister.sch (KiCad schematic (older format))
At the start: 6 parts, among them Q3 BSS138, Q4 BSS138

Commit message: Add files via upload
Parts:
- R5, R6, R7, R8: footprint (none) -> Resistor_SMD:R_0805_2012Metric_Pad1.15x1.40mm_HandSolder
Changed lines of the file:
@@
 EESchema Schematic File Version 4
-LIBS:kicad_master-cache
 EELAYER 30 0
 EELAYER END
 $Descr A4 11693 8268
 encoding utf-8
-Sheet 12 22
+Sheet 12 21
 Title ""
 Date ""
@@
 F 0 "R5" H 3670 3946 50  0000 L CNN
 F 1 "Pull" H 3670 3855 50  0000 L CNN
-F 2 "" V 3530 3900 50  0001 C CNN
+F 2 "Resistor_SMD:R_0805_2012Metric_Pad1.15x1.40mm_HandSolder" V 3530 3900 50  0001 C CNN
 F 3 "~" H 3600 3900 50  0001 C CNN
 	1    3600 3900
@@
 F 0 "R7" H 6920 3896 50  0000 L CNN
 F 1 "Pull" H 6920 3805 50  0000 L CNN
-F 2 "" V 6780 3850 50  0001 C CNN
+F 2 "Resistor_SMD:R_0805_2012Metric_Pad1.15x1.40mm_HandSolder" V 6780 3850 50  0001 C CNN
 F 3 "~" H 6850 3850 50  0001 C CNN
 	1    6850 3850
@@
 F 0 "R6" H 3970 5046 50  0000 L CNN
 F 1 "Pull" H 3970 4955 50  0000 L CNN
-F 2 "" V 3830 5000 50  0001 C CNN
+F 2 "Resistor_SMD:R_0805_2012Metric_Pad1.15x1.40mm_HandSolder" V 3830 5000 50  0001 C CNN
 F 3 "~" H 3900 5000 50  0001 C CNN
 	1    3900 5000
@@
 F 0 "R8" H 7220 5196 50  0000 L CNN
 F 1 "Pull" H 7220 5105 50  0000 L CNN
-F 2 "" V 7080 5150 50  0001 C CNN
+F 2 "Resistor_SMD:R_0805_2012Metric_Pad1.15x1.40mm_HandSolder" V 7080 5150 50  0001 C CNN
 F 3 "~" H 7150 5150 50  0001 C CNN
 	1    7150 5150

Commit message: avancement général du routage
Parts:
- Q3, Q4: symbol Transistor_FET:BSS138 -> shield_etage2-rescue:BSS138-Transistor_FET
- R5, R6, R7, R8: symbol Device:R -> shield_etage2-rescue:R-Device
Changed lines of the file:
@@
 $EndDescr
 $Comp
-L Device:R R?
+L shield_etage2-rescue:R-Device R?
 U 1 1 5E667E37
 P 3600 3900
@@
 $EndComp
 $Comp
-L Device:R R?
+L shield_etage2-rescue:R-Device R?
 U 1 1 5E667E3D
 P 6850 3850
@@
 	2200 4350 3600 4350
 $Comp
-L Transistor_FET:BSS138 Q?
+L shield_etage2-rescue:BSS138-Transistor_FET Q?
 U 1 1 5E667E46
 P 5100 4250
@@
 $EndComp
 $Comp
-L Transistor_FET:BSS138 Q?
+L shield_etage2-rescue:BSS138-Transistor_FET Q?
 U 1 1 5E667E4D
 P 5350 5350
@@
 $EndComp
 $Comp
-L Device:R R?
+L shield_etage2-rescue:R-Device R?
 U 1 1 5E667E56
 P 3900 5000
@@
 	6850 4350 8300 4350
 $Comp
-L Device:R R?
+L shield_etage2-rescue:R-Device R?
 U 1 1 5E667E61
 P 7150 5150
@@
 STM32_CP
 $Comp
-L power:+2V8 #PWR024
+L shield_etage2-rescue:+2V8-power #PWR024
 U 1 1 5E669CBC
 P 3600 3200
@@
 $EndComp
 $Comp
-L power:+3V3 #PWR025
+L shield_etage2-rescue:+3V3-power #PWR025
 U 1 1 5E66B01C
 P 6850 3200
