File: LevelShifter_ToF_I2C.sch (KiCad schematic (older format))
At the start: 6 parts, among them Q1 BSS138, Q2 BSS138

Commit message: Add files via upload
Parts:
- R1, R2, R3, R4: footprint (none) -> Resistor_SMD:R_0805_2012Metric_Pad1.15x1.40mm_HandSolder
Changed lines of the file:
@@
 EESchema Schematic File Version 4
-LIBS:kicad_master-cache
 EELAYER 30 0
 EELAYER END
 $Descr A4 11693 8268
 encoding utf-8
-Sheet 2 22
+Sheet 2 21
 Title ""
 Date ""
@@
 F 0 "R1" H 2720 2196 50  0000 L CNN
 F 1 "Pull" H 2720 2105 50  0000 L CNN
-F 2 "" V 2580 2150 50  0001 C CNN
+F 2 "Resistor_SMD:R_0805_2012Metric_Pad1.15x1.40mm_HandSolder" V 2580 2150 50  0001 C CNN
 F 3 "~" H 2650 2150 50  0001 C CNN
 	1    2650 2150
@@
 F 0 "R3" H 5920 2196 50  0000 L CNN
 F 1 "Pull" H 5920 2105 50  0000 L CNN
-F 2 "" V 5780 2150 50  0001 C CNN
+F 2 "Resistor_SMD:R_0805_2012Metric_Pad1.15x1.40mm_HandSolder" V 5780 2150 50  0001 C CNN
 F 3 "~" H 5850 2150 50  0001 C CNN
 	1    5850 2150
@@
 F 0 "R2" H 2970 3346 50  0000 L CNN
 F 1 "Pull" H 2970 3255 50  0000 L CNN
-F 2 "" V 2830 3300 50  0001 C CNN
+F 2 "Resistor_SMD:R_0805_2012Metric_Pad1.15x1.40mm_HandSolder" V 2830 3300 50  0001 C CNN
 F 3 "~" H 2900 3300 50  0001 C CNN
 	1    2900 3300
@@
 F 0 "R4" H 6220 3296 50  0000 L CNN
 F 1 "Pull" H 6220 3205 50  0000 L CNN
-F 2 "" V 6080 3250 50  0001 C CNN
+F 2 "Resistor_SMD:R_0805_2012Metric_Pad1.15x1.40mm_HandSolder" V 6080 3250 50  0001 C CNN
 F 3 "~" H 6150 3250 50  0001 C CNN
 	1    6150 3250

Commit message: avancement général du routage
Parts:
- Q1, Q2: symbol Transistor_FET:BSS138 -> shield_etage2-rescue:BSS138-Transistor_FET
- R1, R2, R3, R4: symbol Device:R -> shield_etage2-rescue:R-Device
Changed lines of the file:
@@
 I2C_SCL_ToF
 $Comp
-L power:+3.3V #PWR?
+L shield_etage2-rescue:+3.3V-power #PWR?
 U 1 1 5E632CF7
 P 5850 1850
@@
 $EndComp
 $Comp
-L power:+2V8 #PWR?
+L shield_etage2-rescue:+2V8-power #PWR?
 U 1 1 5E632CFD
 P 2650 1850
@@
 $EndComp
 $Comp
-L Device:R R?
+L shield_etage2-rescue:R-Device R?
 U 1 1 5E632D03
 P 2650 2150
@@
 $EndComp
 $Comp
-L Device:R R?
+L shield_etage2-rescue:R-Device R?
 U 1 1 5E632D09
 P 5850 2150
@@
 $EndComp
 $Comp
-L Transistor_FET:BSS138 Q?
+L shield_etage2-rescue:BSS138-Transistor_FET Q?
 U 1 1 5E632D0F
 P 4200 2550
@@
 I2C_SDA_ToF
 $Comp
-L Device:R R?
+L shield_etage2-rescue:R-Device R?
 U 1 1 5E63BCC7
 P 2900 3300
@@
 $EndComp
 $Comp
-L Device:R R?
+L shield_etage2-rescue:R-Device R?
 U 1 1 5E63BCCD
 P 6150 3250
@@
 	1800 3750 2900 3750
 $Comp
-L Transistor_FET:BSS138 Q?
+L shield_etage2-rescue:BSS138-Transistor_FET Q?
 U 1 1 5E63BCD3
 P 4450 3650
