File: f4.sch (KiCad schematic (older format))
At the start: 1 part, among them U1 STM32F401RETx

Commit message: Add files via upload
Parts:
- removed U1: STM32F401RETx, Package_QFP:LQFP-64_10x10mm_P0.5mm, symbol MCU_ST_STM32F4:STM32F401RETx
- added A1: NUCLEO-F401RE, NUCLEO_F401RE:ST_NUCLEO-F401RE, symbol F401RE:NUCLEO-F401RE
- added C10: 1µ, symbol Device:C
- added C5: 100n, symbol Device:C
- added SW1: SW_Push, symbol Switch:SW_Push
Connections:
- net labels added: +5V
- net labels removed: debug_rx, debug_tx
- wire segments 15 -> 11
- no-connect marks 0 -> 69
Other:
- note added: "Broches de la partie "morpho" de la nucleo, qui nous intéressent donc"
- note added: "On rajoute un bouton pour reset la carte\nainsi que le registre à décalage\nComme on la place au-dessus de la f4, \non n'a plus accès au bouton\nreset de la nucleo\n"
- note added: "PA9\nPA10\n"
- note added: "PB12\nPB13\nPB14\nPB15"
- note added: "PB3\nPB4\nPB5\nPB6\n"
- note added: "PB7\n"
- note added: "PC0\nPC1\n"
- note added: "PC6\n"
- note added: "PC7\n"
- note added: "PC8\n"
- note added: "PC9"
- note added: "Tout ça, ce sont les connecteurs Arduino de la F4.\nEn fait, on s'en fiche un peu, mais je les ai placés là pour\nleur donner un peu de visibilité, qu'on voie bien que\ntous les pins de la nucleo sont représentés."

Commit message: Add files via upload
Parts:
- C10, C5: footprint (none) -> Capacitor_SMD:C_0805_2012Metric_Pad1.15x1.40mm_HandSolder
- SW1: footprint (none) -> Button_Switch_SMD:SW_Push_1P1T_NO_6x6mm_H9.5mm
Changed lines of the file:
@@
 EESchema Schematic File Version 4
-LIBS:kicad_master-cache
 EELAYER 30 0
 EELAYER END
 $Descr A3 16535 11693
 encoding utf-8
-Sheet 22 22
+Sheet 21 21
 Title ""
 Date ""
@@
 F 0 "C5" H 14415 2296 50  0000 L CNN
 F 1 "100n" H 14415 2205 50  0000 L CNN
-F 2 "" H 14338 2100 50  0001 C CNN
+F 2 "Capacitor_SMD:C_0805_2012Metric_Pad1.15x1.40mm_HandSolder" H 14338 2100 50  0001 C CNN
 F 3 "~" H 14300 2250 50  0001 C CNN
 	1    14300 2250
@@
 F 0 "SW1" V 13846 2152 50  0000 R CNN
 F 1 "SW_Push" V 13755 2152 50  0000 R CNN
-F 2 "" H 13800 2400 50  0001 C CNN
+F 2 "Button_Switch_SMD:SW_Push_1P1T_NO_6x6mm_H9.5mm" H 13800 2400 50  0001 C CNN
 F 3 "~" H 13800 2400 50  0001 C CNN
 	1    13800 2200
@@
 F 0 "C10" V 5602 3200 50  0000 C CNN
 F 1 "1µ" V 5511 3200 50  0000 C CNN
-F 2 "" H 5388 3050 50  0001 C CNN
+F 2 "Capacitor_SMD:C_0805_2012Metric_Pad1.15x1.40mm_HandSolder" H 5388 3050 50  0001 C CNN
 F 3 "~" H 5350 3200 50  0001 C CNN
 	1    5350 3200

Commit message: avancement général du routage
Parts:
- A1: symbol F401RE:NUCLEO-F401RE -> shield_etage2-rescue:NUCLEO-F401RE-F401RE
- C10, C5: symbol Device:C -> shield_etage2-rescue:C-Device
- SW1: symbol Switch:SW_Push -> shield_etage2-rescue:SW_Push-Switch
Changed lines of the file:
@@
 NRST
 $Comp
-L Device:C C?
+L shield_etage2-rescue:C-Device C?
 U 1 1 5E81E95C
 P 14300 2250
@@
 $EndComp
 $Comp
-L power:GND #PWR?
+L shield_etage2-rescue:GND-power #PWR?
 U 1 1 5E81E962
 P 14300 2400
@@
 $EndComp
 $Comp
-L power:GND #PWR?
+L shield_etage2-rescue:GND-power #PWR?
 U 1 1 5E81E968
 P 13800 2400
@@
 $EndComp
 $Comp
-L Switch:SW_Push SW1
+L shield_etage2-rescue:SW_Push-Switch SW1
 U 1 1 5E823FD4
 P 13800 2200
@@
 Connection ~ 13800 1950
 $Comp
-L F401RE:NUCLEO-F401RE A1
+L shield_etage2-rescue:NUCLEO-F401RE-F401RE A1
 U 1 1 5E889489
 P 3650 4500
@@
 $EndComp
 $Comp
-L F401RE:NUCLEO-F401RE A1
+L shield_etage2-rescue:NUCLEO-F401RE-F401RE A1
 U 2 1 5E88AFC4
 P 7500 4600
@@
 I2C_ToF_SDA
 $Comp
-L F401RE:NUCLEO-F401RE A1
+L shield_etage2-rescue:NUCLEO-F401RE-F401RE A1
 U 3 1 5E88FA35
 P 11950 5000
@@
 PB7\n
 $Comp
-L power:+5V #PWR0126
+L shield_etage2-rescue:+5V-power #PWR0126
 U 1 1 5E8EEA6E
 P 5050 3150
@@
 $EndComp
 $Comp
-L Device:C C10
+L shield_etage2-rescue:C-Device C10
 U 1 1 5E8F04FC
 P 5350 3200
@@
 $EndComp
 $Comp
-L power:GND #PWR0127
+L shield_etage2-rescue:GND-power #PWR0127
 U 1 1 5E8F1C24
 P 5500 3200
@@
 Connection ~ 5050 3200
 $Comp
-L power:GND #PWR0128
+L shield_etage2-rescue:GND-power #PWR0128
 U 1 1 5E8F67E4
 P 4350 6100
@@
 $EndComp
 $Comp
-L power:GND #PWR0131
+L shield_etage2-rescue:GND-power #PWR0131
 U 1 1 5E8F7826
 P 8200 6200
@@
 Connection ~ 8200 6100
 $Comp
-L F401RE:NUCLEO-F401RE A1
+L shield_etage2-rescue:NUCLEO-F401RE-F401RE A1
 U 6 1 5E8F8F98
 P 13800 4950
@@
 $EndComp
 $Comp
-L power:GND #PWR0132
+L shield_etage2-rescue:GND-power #PWR0132
 U 1 1 5E8FE2BA
 P 14400 5550
@@
 $EndComp
 $Comp
-L power:GND #PWR0133
+L shield_etage2-rescue:GND-power #PWR0133
 U 1 1 5E8FEF08
 P 12550 5400
@@
 $EndComp
 $Comp
-L F401RE:NUCLEO-F401RE A1
+L shield_etage2-rescue:NUCLEO-F401RE-F401RE A1
 U 4 1 5E90550E
 P 12300 6350
@@
 $EndComp
 $Comp
-L F401RE:NUCLEO-F401RE A1
+L shield_etage2-rescue:NUCLEO-F401RE-F401RE A1
 U 5 1 5E908B54
 P 13800 6400
@@
 NoConn ~ 11900 5950
 $Comp
-L power:+3V3 #PWR0134
+L shield_etage2-rescue:+3V3-power #PWR0134
 U 1 1 5E93C2F8
 P 4650 2950
@@
 	4650 3000 4650 2950
 $Comp
-L power:PWR_FLAG #FLG0102
+L shield_etage2-rescue:PWR_FLAG-power #FLG0102
 U 1 1 5E94097F
 P 4350 3000
