File: moteur_conn.sch (KiCad schematic (older format))
At the start: 1 part, among them J12 Conn_01x02

Commit message: Add files via upload
Parts:
- J12: value Conn_01x02 -> Moteur; footprint (none) -> Connector_JST:JST_PH_B2B-PH-K_1x02_P2.00mm_Vertical
Changed lines of the file:
@@
 EESchema Schematic File Version 4
-LIBS:kicad_master-cache
 EELAYER 30 0
 EELAYER END
 $Descr A4 11693 8268
 encoding utf-8
-Sheet 14 22
+Sheet 15 21
 Title ""
 Date ""
@@
 AR Path="/5E685B22/5E6C3064" Ref="J12"  Part="1"
 AR Path="/5E685A03/5E6C3064" Ref="J11"  Part="1"
-F 0 "J11" H 5530 2592 50  0000 L CNN
-F 1 "Conn_01x02" H 5530 2501 50  0000 L CNN
-F 2 "" H 5450 2600 50  0001 C CNN
+F 0 "J12" H 5530 2592 50  0000 L CNN
+F 1 "Moteur" H 5530 2501 50  0000 L CNN
+F 2 "Connector_JST:JST_PH_B2B-PH-K_1x02_P2.00mm_Vertical" H 5450 2600 50  0001 C CNN
 F 3 "~" H 5450 2600 50  0001 C CNN
 	1    5450 2600

Commit message: avancement général du routage
Parts:
- J12: symbol Connector_Generic:Conn_01x02 -> shield_etage2-rescue:Conn_01x02-Connector_Generic
Changed lines of the file:
@@
 	5250 2700 4800 2700
 $Comp
-L Connector_Generic:Conn_01x02 J12
+L shield_etage2-rescue:Conn_01x02-Connector_Generic J12
 U 1 1 5E6C3064
 P 5450 2600
