File: regulateur.sch (KiCad schematic (older format))
At the start: 10 parts, among them U3 LM317_TO3, U4 LM317_TO3

Commit message: avancement général du routage
Parts:
- C1, C2, C8, C9: symbol Device:C -> shield_etage2-rescue:C-Device
- R10, R16, R17, R9: symbol Device:R -> shield_etage2-rescue:R-Device
- U3, U4: symbol Regulator_Linear:LM317_TO3 -> shield_etage2-rescue:LM317_TO3-Regulator_Linear
Changed lines of the file:
@@
 $EndDescr
 $Comp
-L power:+2V8 #PWR028
+L shield_etage2-rescue:+2V8-power #PWR028
 U 1 1 5E67A02D
 P 8700 3650
@@
 $EndComp
 $Comp
-L Regulator_Linear:LM317_TO3 U4
+L shield_etage2-rescue:LM317_TO3-Regulator_Linear U4
 U 1 1 5E846C10
 P 3150 3650
@@
 	2350 3650 2650 3650
 $Comp
-L Device:R R16
+L shield_etage2-rescue:R-Device R16
 U 1 1 5E846C17
 P 3600 3950
@@
 $EndComp
 $Comp
-L Device:R R17
+L shield_etage2-rescue:R-Device R17
 U 1 1 5E846C1D
 P 3600 4400
@@
 $EndComp
 $Comp
-L Device:C C9
+L shield_etage2-rescue:C-Device C9
 U 1 1 5E846C23
 P 4150 4150
@@
 $EndComp
 $Comp
-L Device:C C8
+L shield_etage2-rescue:C-Device C8
 U 1 1 5E846C29
 P 2650 4200
@@
 	3600 4150 3600 4250
 $Comp
-L power:GND #PWR0108
+L shield_etage2-rescue:GND-power #PWR0108
 U 1 1 5E846C41
 P 3200 4800
@@
 	8200 3650 8700 3650
 $Comp
-L Device:R R10
+L shield_etage2-rescue:R-Device R10
 U 1 1 5E67CD58
 P 7650 4400
@@
 Connection ~ 7250 4800
 $Comp
-L power:GND #PWR027
+L shield_etage2-rescue:GND-power #PWR027
 U 1 1 5E67EDD3
 P 7250 4800
@@
 	6700 4050 6700 3650
 $Comp
-L Device:C C1
+L shield_etage2-rescue:C-Device C1
 U 1 1 5E67DD37
 P 6700 4200
@@
 $EndComp
 $Comp
-L Device:C C2
+L shield_etage2-rescue:C-Device C2
 U 1 1 5E67D126
 P 8200 4150
@@
 $EndComp
 $Comp
-L Device:R R9
+L shield_etage2-rescue:R-Device R9
 U 1 1 5E8486F2
 P 7650 3950
@@
 $EndComp
 $Comp
-L Regulator_Linear:LM317_TO3 U3
+L shield_etage2-rescue:LM317_TO3-Regulator_Linear U3
 U 1 1 5E677609
 P 7200 3650
@@
 $EndComp
 $Comp
-L power:+5V #PWR0120
+L shield_etage2-rescue:+5V-power #PWR0120
 U 1 1 5E8571A1
 P 5250 3650
@@
 	5250 3650 6700 3650
 $Comp
-L power:+6V #PWR?
+L shield_etage2-rescue:+6V-power #PWR?
 U 1 1 5E860379
 P 2350 3650
