File: shield_etage2.sch (KiCad schematic (older format))
At the start: 8 parts, among them J1 Conn_01x02, J2 Conn_01x02

Commit message: avancement général du routage
Parts:
- C3, C4: symbol Device:C -> shield_etage2-rescue:C-Device
- H1, H2, H3, H4: symbol Mechanical:MountingHole_Pad -> shield_etage2-rescue:MountingHole_Pad-Mechanical
- J1, J2: symbol Connector_Generic:Conn_01x02 -> shield_etage2-rescue:Conn_01x02-Connector_Generic
Changed lines of the file:
@@
 $EndSheet
 $Comp
-L Connector_Generic:Conn_01x02 J1
+L shield_etage2-rescue:Conn_01x02-Connector_Generic J1
 U 1 1 5E6A42B0
 P 6300 2350
@@
 $EndComp
 $Comp
-L power:GND #PWR03
+L shield_etage2-rescue:GND-power #PWR03
 U 1 1 5E6A7F5C
 P 8100 3150
@@
 $EndComp
 $Comp
-L Connector_Generic:Conn_01x02 J2
+L shield_etage2-rescue:Conn_01x02-Connector_Generic J2
 U 1 1 5E6A5692
 P 7850 2350
@@
 ALIM_MOTEURS
 $Comp
-L power:GND #PWR02
+L shield_etage2-rescue:GND-power #PWR02
 U 1 1 5E6A6CBF
 P 6500 3150
@@
 	7950 2550 8100 2550
 $Comp
-L power:PWR_FLAG #FLG01
+L shield_etage2-rescue:PWR_FLAG-power #FLG01
 U 1 1 5E6C9FE5
 P 6300 3050
@@
 $EndComp
 $Comp
-L Device:C C3
+L shield_etage2-rescue:C-Device C3
 U 1 1 5E6A8F61
 P 6050 2750
@@
 $EndComp
 $Comp
-L Device:C C4
+L shield_etage2-rescue:C-Device C4
 U 1 1 5E6AD189
 P 7600 2750
@@
 $EndComp
 $Comp
-L power:GND #PWR0101
+L shield_etage2-rescue:GND-power #PWR0101
 U 1 1 5E6ADDFF
 P 7450 2750
@@
 $EndComp
 $Comp
-L power:GND #PWR0102
+L shield_etage2-rescue:GND-power #PWR0102
 U 1 1 5E6AE41B
 P 5900 2750
@@
 	10750 4600 11800 4600
 $Comp
-L Mechanical:MountingHole_Pad H1
+L shield_etage2-rescue:MountingHole_Pad-Mechanical H1
 U 1 1 5E81B7D6
 P 14800 2250
@@
 $EndComp
 $Comp
-L Mechanical:MountingHole_Pad H2
+L shield_etage2-rescue:MountingHole_Pad-Mechanical H2
 U 1 1 5E81C6C2
 P 14800 2450
@@
 $EndComp
 $Comp
-L Mechanical:MountingHole_Pad H3
+L shield_etage2-rescue:MountingHole_Pad-Mechanical H3
 U 1 1 5E81F44B
 P 14800 2650
@@
 $EndComp
 $Comp
-L Mechanical:MountingHole_Pad H4
+L shield_etage2-rescue:MountingHole_Pad-Mechanical H4
 U 1 1 5E81F451
 P 14800 2850
@@
 	14700 2850 14700 3000
 $Comp
-L power:GND #PWR0103
+L shield_etage2-rescue:GND-power #PWR0103
 U 1 1 5E82CE64
 P 14700 3000
@@
 Connection ~ 6500 3050
 $Comp
-L power:PWR_FLAG #FLG02
+L shield_etage2-rescue:PWR_FLAG-power #FLG02
 U 1 1 5E6CC857
 P 6500 3050
@@
 	7850 2750 7850 3050
 $Comp
-L power:PWR_FLAG #FLG0103
+L shield_etage2-rescue:PWR_FLAG-power #FLG0103
 U 1 1 5E95264E
 P 7850 3050
@@
 $EndSheet
 $Comp
-L power:+6V #PWR0105
+L shield_etage2-rescue:+6V-power #PWR0105
 U 1 1 5E859DB4
 P 6300 3150
